File: qeqeqwe/qeqeqwe.kicad_pcb (KiCad board)
At the start: 2 copper layers, 11 parts, among them J1 USB_A, J2 USB_A, U1 ATtiny85-20S

Commit message: dgdgegergregre
Parts:
- added U2: USB_A, Connector_USB:USB_A_Receptacle_GCT_USB1046, F.Cu at (154.9, 76.2)
- J1, J2: value USB_A -> Conn_01x04; footprint Connector_USB:USB_A_Receptacle_GCT_USB1046 -> Connector_PinHeader_2.54mm:PinHeader_1x04_P2.54mm_Vertical
- moved J1 97.7 mm to (91.4, 64.7), turned to 0 degrees
- moved J2 85.5 mm to (101.6, 58.4), turned to 0 degrees
- moved R1 63.0 mm to (102.6, 81.3), turned to 90 degrees
- moved D1 58.9 mm to (106.7, 83.8), turned to -90 degrees
- moved D2 56.6 mm to (114.6, 84.9)
- moved C1 46.4 mm to (125.4, 83.8)
- moved U1 45.5 mm to (111.8, 73.7)
- moved R2 45.1 mm to (120.1, 79.0)
- moved D3 38.5 mm to (134.6, 61.0)
- moved R3 37.8 mm to (120.1, 82.0)
- moved R4 28.9 mm to (120.1, 84.9)
Connections:
- D1 pad 1: Net-(D1-K) -> +5V
- J1 pad 1: Net-(J1-VBUS) -> Net-(J1-Pin_1)
- J1 pad 2: Net-(J1-D-) -> Net-(J1-Pin_2)
- J1 pad 3: Net-(J1-D+) -> Net-(J1-Pin_3)
- J1 pad 4: +5V -> GND
- J2 pad 1: Net-(J2-VBUS) -> Net-(J2-Pin_1)
- J2 pad 2: Net-(J2-D-) -> Net-(J2-Pin_2)
- J2 pad 3: Net-(J2-D+) -> Net-(J2-Pin_3)
- J2 pad 4: GND -> +5V
- R1 pad 1: Net-(D1-K) -> +5V
- R1 pad 2: Net-(J2-D+) -> Net-(J1-Pin_3)
- R2 pad 2: Net-(J2-D-) -> Net-(J1-Pin_2)
- R3 pad 2: Net-(J1-D-) -> Net-(J2-Pin_2)
- U1 pad 1: Net-(J2-VBUS) -> Net-(J1-Pin_1)
- U1 pad 2: Net-(J2-D-) -> Net-(J1-Pin_2)
- U1 pad 3: Net-(J2-D+) -> Net-(J1-Pin_3)
- U1 pad 5: Net-(J1-VBUS) -> Net-(J2-Pin_1)
- U1 pad 6: Net-(J1-D-) -> Net-(J2-Pin_2)
- U1 pad 7: Net-(J1-D+) -> Net-(J2-Pin_3)

Commit message: bkbbj
Parts:
- moved J1 67.9 mm to (159.3, 65.8), turned to 90 degrees
- moved J2 59.9 mm to (159.0, 75.6), turned to 90 degrees
- moved R3 57.0 mm to (174.7, 66.0)
- moved R1 52.5 mm to (153.7, 69.4), turned to 0 degrees
- moved U1 52.3 mm to (164.0, 70.7), turned to 180 degrees
- moved D3 42.9 mm to (174.9, 75.9), turned to 90 degrees
- moved D1 41.0 mm to (143.8, 66.5), turned to 90 degrees
- moved D2 37.5 mm to (148.0, 67.7), turned to -90 degrees
- moved R2 34.1 mm to (153.7, 73.5)
- moved R4 30.2 mm to (148.8, 75.5), turned to -90 degrees
- moved U2 23.4 mm to (132.1, 71.1), turned to -90 degrees
- moved C1 20.8 mm to (144.4, 75.3), turned to 90 degrees
Connections:
- D1 pad 1: +5V -> Net-(D1-K)
- R1 pad 1: +5V -> Net-(D1-K)
- U2 pad 3: +5V -> Net-(D1-K)
Routing:
- net GND: track 0.00 -> 70.1 mm
- net Net-(J2-Pin_2): track 0.00 -> 42.7 mm
- net +5V: track 0.00 -> 40.9 mm, vias 0 -> 6
- net Net-(D2-K): track 0.00 -> 24.4 mm, vias 0 -> 2
- net Net-(J1-Pin_3): track 0.00 -> 22.9 mm, vias 0 -> 3
- net Net-(D1-K): track 0.00 -> 15.6 mm, vias 0 -> 2
- net Net-(J2-Pin_1): track 0.00 -> 13.4 mm, vias 0 -> 1
- net Net-(J1-Pin_1): track 0.00 -> 11.1 mm
- net Net-(J1-Pin_2): track 0.00 -> 8.74 mm
- net Net-(D3-A): track 0.00 -> 7.81 mm
- net Net-(J2-Pin_3): track 0.00 -> 6.24 mm
- added copper zone on F.Cu, net (none)
Other:
- board outline added: 52.5 x 15.2 mm
