File: 3. ročník/13.10.2025/13.10.2025.kicad_sch (KiCad schematic)
At the start: 2 parts

Commit message: rwrwerwer
Parts:
- removed S3: Vol-, Button_Switch_THT:SW_PUSH_6mm, symbol PCM_SL_Devices:Push_Button
- removed S4: Vol+, Button_Switch_THT:SW_PUSH_6mm, symbol PCM_SL_Devices:Push_Button
- added C1, C10, C12, C13, C2, C3, C6, C9: C, symbol Device:C
- added C11, C14, C4, C5, C7, C8: C_Polarized, symbol Device:C_Polarized
- added J1: Barrel_Jack, Connector_BarrelJack:BarrelJack_SwitchcraftConxall_RAPC10U_Horizontal, symbol Connector:Barrel_Jack
- added R1, R2, R3, R4, R5: R, symbol Device:R
- added RDA5807FP1: ~, symbol ICs:RDA5807FP
- added SW1: SW_SPST, symbol Switch:SW_SPST
- added TDA_1: ~, symbol ICs:TDA2822
