File: 3. ročník/13.10.2025/13.10.2025.kicad_sch (KiCad schematic)
At the start: 30 parts, among them J1 Barrel_Jack, SW1 SW_SPST

Commit message: weqwe
Parts:
- removed J1: Barrel_Jack, Connector_BarrelJack:BarrelJack_SwitchcraftConxall_RAPC10U_Horizontal, symbol Connector:Barrel_Jack
- removed TDA_1: ~, symbol ICs:TDA2822
- added BT1: Battery, symbol Device:Battery
- added C15: 104, symbol Device:C
- added J1: Barrel_Jack_Switch, Connector_BarrelJack:BarrelJack_CUI_PJ-102AH_Horizontal, symbol Connector:Barrel_Jack_Switch
- added LS1: Speaker, symbol Device:Speaker
- added R6: 2K, symbol Device:R
- added SW2: CH-, symbol Switch:SW_Push
- added SW3: Vol-, symbol Switch:SW_Push
- added SW4: Vol+, symbol Switch:SW_Push
- added SW5: CH+, symbol Switch:SW_Push
- added TDA2822: ~, symbol ICs:TDA2822
- added Y1: 32.768K, symbol Device:Crystal
- C1, C10: value C -> 103
- C11, C8: value C_Polarized -> 10U
- C12, C13, C6: value C -> 104
- C14: value C_Polarized -> 1000U
- C2: value C -> 102
- C3: value C -> 223
- C4, C5: value C_Polarized -> 100U
- C7: value C_Polarized -> 470U
- C9: value C -> 222
- D1: value D_Zener -> 3.3V
- D3: value D -> 1N4007
- L1: value L -> 0, 1
- L2, L3: value L -> 1UH
- R1, R2: value R -> 10K
- R3: value R -> 22
- R4, R5: value R -> 2.2
Connections:
- net GND: now also C1.2, C10.2, C3.1, C9.2, D1.2 (A), L1.1, R1.2, R2.2, RDA5807FP1.11 (GND), RDA5807FP1.14 (GND), RDA5807FP1.2 (GND), RDA5807FP1.3 (RF_GND), RDA5807FP1.5 (GND), SW1.1 (A), SW2.1, SW3.2, SW4.2, SW5.1, TDA2822.4, TDA2822.6, Y1.1
- net at C2.1: now also RDA5807FP1.4 (FMIN)
- net at C2.2: now also AE1.1 (A), L1.2
- net at L2.1: now also RDA5807FP1.12 (ROUT)
- net at L2.2: now also C5.1
- net at R4.1: now also LS1.2, TDA2822.1
- net at R4.2: now also C13.1
- net at C6.1: now also C3.2, C7.1, D1.1 (K), R3.1, RDA5807FP1.10 (VDD), RDA5807FP1.6 (GND)
- net 0: now reaches C6.2
- net 0: now also C12.2, C13.2, C14.2, C7.2, C15.2
- net at C11.1: now also TDA2822.8
- net at C11.2: now also C10.1, TDA2822.5
- net at R2.1: now also C8.2, C9.1, TDA2822.7
- net at R3.2: now also C14.1, D3.1 (K), BT1.1 (+), C15.1, TDA2822.2
- net at C5.2: now also C4.2, C8.1, R1.1
- net at D2.1 (K): now also SW1.2 (B), BT1.2 (-)
- net at D2.2 (A): now also R6.2
- net at C4.1: now also L3.2
- net at RDA5807FP1.1 (GPIO1): now also C1.1
- net at RDA5807FP1.15 (GPIO3): now also SW3.1
- net at RDA5807FP1.16 (GPIO2): now also SW4.1
- net at RDA5807FP1.7 (SCLK): now also SW2.2
- net at RDA5807FP1.8 (SDA): now also SW5.2
- net at RDA5807FP1.9 (RCLK): now also Y1.2
- net at C12.1: now also R5.2
- net at R5.1: now also LS1.1, TDA2822.3
- net at D3.2 (A): now also R6.1
- net at L3.1: now also RDA5807FP1.13 (LOUT)
Other:
- moved on the sheet: AE1, C1, C10, C11, C13, C14, C2, C3, C4, C5, C6, C7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

Commit message: Hello
Parts:
- BT1: value Battery -> 1&650 3.7V

Commit message: jasdfds
Connections:
- net GND: no longer C1.2, C10.2, C3.1, C9.2, D1.2 (A), L1.1, R1.2, R2.2, RDA5807FP1.11 (GND), RDA5807FP1.14 (GND), RDA5807FP1.2 (GND), RDA5807FP1.3 (RF_GND), RDA5807FP1.5 (GND), SW1.1 (A), SW2.1, SW3.2, SW4.2, SW5.1, TDA2822.4, TDA2822.6, Y1.1
- new net Earth: C1.2, C10.2, C3.1, C9.2, D1.2 (A), L1.1, R1.2, R2.2, RDA5807FP1.11 (GND), RDA5807FP1.14 (GND), RDA5807FP1.2 (GND), RDA5807FP1.3 (RF_GND), RDA5807FP1.5 (GND), SW1.1 (A), SW2.1, SW3.2, SW4.2, SW5.1, TDA2822.4, TDA2822.6, Y1.1
Other:
- moved on the sheet: J1

Commit message: ae
Parts:
- BT1: value 1&650 3.7V -> 18650 3.7V
- C1, C10, C11, C12, C13, C14, C15, C2, C3, C4, C5, C6, C7, C8, C9: footprint (none) -> Capacitor_THT:CP_Radial_D5.0mm_P2.50mm
- D2: footprint (none) -> LED_THT:LED_D5.0mm
- R1, R2, R3, R4, R5, R6: footprint (none) -> Resistor_THT:R_Axial_DIN0207_L6.3mm_D2.5mm_P10.16mm_Horizontal
Connections:
- net at BT1.2 (-), D2.1 (K), SW1.2 (B): now also J1.2
- net at J1.1: now also D3.2 (A), R6.1
Changed lines of the file:
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@@
 	)
 	(junction
+		(at 248.92 80.01)
+		(diameter 0)
+		(color 0 0 0 0)
+	)
+	(junction
 		(at 193.04 100.33)
 		(diameter 0)
@@
 	)
 	(junction
+		(at 248.92 100.33)
+		(diameter 0)
+		(color 0 0 0 0)
+	)
+	(junction
 		(at 165.1 100.33)
 		(diameter 0)
@@
 	(wire
 		(pts
+			(xy 248.92 100.33) (xy 259.08 100.33)
+		)
+		(stroke
+			(width 0)
+			(type default)
+		)
+	)
+	(wire
+		(pts
 			(xy 209.55 49.53) (xy 203.2 49.53)
 		)
@@
 	(wire
 		(pts
+			(xy 248.92 80.01) (xy 259.08 80.01)
+		)
+		(stroke
+			(width 0)
+			(type default)
+		)
+	)
+	(wire
+		(pts
 			(xy 143.51 59.69) (xy 162.56 59.69)
 		)
@@
 	(wire
 		(pts
+			(xy 259.08 85.09) (xy 259.08 100.33)
+		)
+		(stroke
+			(width 0)
+			(type default)
+		)
+	)
+	(wire
+		(pts
 			(xy 220.98 100.33) (xy 248.92 100.33)
 		)
@@
 			)
 		)
-		(property "Footprint" ""
+		(property "Footprint" "Capacitor_THT:CP_Radial_D5.0mm_P2.50mm"
 			(at 107.6452 95.25 0)
 			(effects
@@
 	)
 	(symbol
-		(lib_id "PCM_4ms_Power-symbol:GND")
-		(at 39.37 25.4 0)
-		(unit 1)
-		(exclude_from_sim no)
-		(in_bom yes)
-		(on_board yes)
-		(dnp no)
-		(fields_autoplaced yes)
-		(property "Reference" "#PWR013"
-			(at 39.37 31.75 0)
-			(effects
-				(font
-					(size 1.27 1.27)
-				)
-				(hide yes)
-			)
-		)
-		(property "Value" "GND"
-			(at 39.37 30.48 0)
-			(effects
-				(font
-					(size 1.27 1.27)
-				)
-			)
-		)
-		(property "Footprint" ""
-			(at 39.37 25.4 0)
-			(effects
-				(font
-					(size 1.27 1.27)
-				)
-				(hide yes)
-			)
-		)
-		(property "Datasheet" ""
-			(at 39.37 25.4 0)
-			(effects
-				(font
-					(size 1.27 1.27)
-				)
-				(hide yes)
-			)
-		)
-		(property "Description" ""
-			(at 39.37 25.4 0)
-			(effects
-				(font
-					(size 1.27 1.27)
-				)
-			)
-		)
-		(pin "1"
-		)
-		(instances
-			(project "13.10.2025"
-				(path "/7c5a3e52-8d09-4d48-8225-83045c852ee9"
-					(reference "#PWR013")
-					(unit 1)
-				)
-			)
-		)
-	)
-	(symbol
 		(lib_id "Device:L")
 		(at 119.38 39.37 90)
@@
 			)
 		)
-		(property "Footprint" ""
+		(property "Footprint" "Resistor_THT:R_Axial_DIN0207_L6.3mm_D2.5mm_P10.16mm_Horizontal"
 			(at 207.772 59.69 90)
 			(effects
@@
 			)
 		)
-		(property "Footprint" ""
+		(property "Footprint" "Capacitor_THT:CP_Radial_D5.0mm_P2.50mm"
 			(at 144.4752 67.31 0)
 			(effects
@@
 			)
 		)
-		(property "Footprint" ""
+		(property "Footprint" "Capacitor_THT:CP_Radial_D5.0mm_P2.50mm"
 			(at 194.31 78.4352 0)
 			(effects
@@
 			)
 		)
-		(property "Footprint" ""
+		(property "Footprint" "Resistor_THT:R_Axial_DIN0207_L6.3mm_D2.5mm_P10.16mm_Horizontal"
 			(at 176.022 85.09 90)
 			(effects
@@
 			)
 		)
-		(property "Footprint" ""
+		(property "Footprint" "Resistor_THT:R_Axial_DIN0207_L6.3mm_D2.5mm_P10.16mm_Horizontal"
 			(at 166.37 34.798 90)
 			(effects
@@
 			)
 		)
-		(property "Footprint" ""
+		(property "Footprint" "Capacitor_THT:CP_Radial_D5.0mm_P2.50mm"
 			(at 177.4952 43.18 0)
 			(effects
@@
 			)
 		)
-		(property "Value" "1&650 3.7V"
+		(property "Value" "18650 3.7V"
 			(at 224.79 90.8684 0)
 			(effects
@@
 		(on_board yes)
 		(dnp no)
-		(fields_autoplaced yes)
 		(property "Reference" "RDA5807FP1"
-			(at 124.46 74.93 0)
+			(at 107.95 74.93 0)
 			(effects
 				(font
@@
 			)
 		)
-		(property "Footprint" ""
+		(property "Footprint" "Capacitor_THT:CP_Radial_D5.0mm_P2.50mm"
 			(at 134.62 38.4048 0)
 			(effects
@@
 			)
 		)
-		(property "Footprint" ""
+		(property "Footprint" "Capacitor_THT:CP_Radial_D5.0mm_P2.50mm"
 			(at 163.83 75.8952 0)
 			(effects
@@
 			)
 		)
-		(property "Footprint" ""
+		(property "Footprint" "Capacitor_THT:CP_Radial_D5.0mm_P2.50mm"
 			(at 166.0652 88.9 0)
 			(effects
@@
 			)
 		)
-		(property "Footprint" ""
+		(property "Footprint" "LED_THT:LED_D5.0mm"
 			(at 248.92 93.98 0)
 			(effects
@@
 			)
 		)
-		(property "Footprint" ""
+		(property "Footprint" "Capacitor_THT:CP_Radial_D5.0mm_P2.50mm"
 			(at 134.62 32.0548 0)
 			(effects
@@
 			)
 		)
-		(property "Footprint" ""
+		(property "Footprint" "Capacitor_THT:CP_Radial_D5.0mm_P2.50mm"
 			(at 163.5252 67.31 0)
 			(effects
@@
 			)
 		)
-		(property "Footprint" ""
+		(property "Footprint" "Capacitor_THT:CP_Radial_D5.0mm_P2.50mm"
 			(at 215.5952 43.18 0)
 			(effects
@@
 			)
 		)
-		(property "Footprint" ""
+		(property "Footprint" "Capacitor_THT:CP_Radial_D5.0mm_P2.50mm"
 			(at 204.1652 50.8 0)
 			(effects
@@
 			)
 		)
-		(property "Footprint" ""
+		(property "Footprint" "Resistor_THT:R_Axial_DIN0207_L6.3mm_D2.5mm_P10.16mm_Horizontal"
 			(at 201.422 39.37 90)
 			(effects
@@
 			)
 		)
-		(property "Footprint" ""
+		(property "Footprint" "Resistor_THT:R_Axial_DIN0207_L6.3mm_D2.5mm_P10.16mm_Horizontal"
 			(at 148.082 78.74 90)
 			(effects
@@
 			)
 		)
-		(property "Footprint" ""
+		(property "Footprint" "Capacitor_THT:CP_Radial_D5.0mm_P2.50mm"
 			(at 121.92 58.7248 0)
 			(effects
@@
 			)
 		)
-		(property "Footprint" ""
+		(property "Footprint" "Capacitor_THT:CP_Radial_D5.0mm_P2.50mm"
 			(at 96.2152 99.06 0)
 			(effects
@@
 			)
 		)
-		(property "Footprint" ""
+		(property "Footprint" "Resistor_THT:R_Axial_DIN0207_L6.3mm_D2.5mm_P10.16mm_Horizontal"
 			(at 247.142 83.82 90)
 			(effects
@@
 			)
 		)
-		(property "Footprint" ""
+		(property "Footprint" "Capacitor_THT:CP_Radial_D5.0mm_P2.50mm"
 			(at 210.5152 73.66 0)
 			(effects
@@
 			)
 		)
-		(property "Footprint" ""
+		(property "Footprint" "Capacitor_THT:CP_Radial_D5.0mm_P2.50mm"
 			(at 191.4652 88.9 0)
 			(effects

Commit message: ajsd
Parts:
- removed C12: 104, Capacitor_THT:CP_Radial_D5.0mm_P2.50mm, symbol Device:C
- removed TDA2822: ~, symbol ICs:TDA2822
- added C12: 104, Capacitor_THT:CP_Radial_D5.0mm_P2.50mm, symbol Device:C_Small
- added D4: LED1, LED_THT:LED_D3.0mm, symbol Device:LED
- added R6: 10K, Resistor_THT:R_Axial_DIN0207_L6.3mm_D2.5mm_P7.62mm_Horizontal, symbol Device:R
- added TDA2822IC1: ~, Package_DIP:DIP-8_W7.62mm_Socket, symbol ICs:TDA2822
- AE1: footprint (none) -> Connector_Wire:SolderWire-0.1sqmm_1x01_D0.4mm_OD1mm
- BT1: footprint (none) -> Battery:BatteryHolder_Keystone_2460_1xAA
- D2: value LED -> LED2; footprint LED_THT:LED_D5.0mm -> LED_THT:LED_D3.0mm
- R1, R4: footprint Resistor_THT:R_Axial_DIN0207_L6.3mm_D2.5mm_P10.16mm_Horizontal -> Resistor_THT:R_Axial_DIN0207_L6.3mm_D2.5mm_P7.62mm_Horizontal
- R10: renamed from R6; footprint Resistor_THT:R_Axial_DIN0207_L6.3mm_D2.5mm_P10.16mm_Horizontal -> Resistor_THT:R_Axial_DIN0207_L6.3mm_D2.5mm_P7.62mm_Horizontal
- R2: renamed from R3; footprint Resistor_THT:R_Axial_DIN0207_L6.3mm_D2.5mm_P10.16mm_Horizontal -> Resistor_THT:R_Axial_DIN0207_L6.3mm_D2.5mm_P7.62mm_Horizontal
- R3: renamed from R2; footprint Resistor_THT:R_Axial_DIN0207_L6.3mm_D2.5mm_P10.16mm_Horizontal -> Resistor_THT:R_Axial_DIN0207_L6.3mm_D2.5mm_P7.62mm_Horizontal
- R5: value 2.2 -> 2k2; footprint Resistor_THT:R_Axial_DIN0207_L6.3mm_D2.5mm_P10.16mm_Horizontal -> Resistor_THT:R_Axial_DIN0207_L6.3mm_D2.5mm_P7.62mm_Horizontal
- RDA5807FP1: footprint (none) -> Package_DIP:DIP-16_W8.89mm_SMDSocket_LongPads
- renumbered SW1 to K1, SW2 to S1, SW5 to S2, D1 to Z1
Connections:
- net Earth: no longer C1.2, C10.2, C3.1, C9.2, K1.1 (A), L1.1, R1.2, R3.2, RDA5807FP1.11 (GND), RDA5807FP1.14 (GND), S1.1, S2.1, SW3.2, SW4.2, Y1.1, Z1.2 (A)
- net at LS1.2, R4.1: now also TDA2822IC1.1
- net at C3.2, C6.1, C7.1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: now also R6.2; no longer R2.1
- net at LS1.1, R5.1: now also TDA2822IC1.3
- net at C11.1: now also TDA2822IC1.8
- net at C10.1, C11.2: now also TDA2822IC1.5
- net at C8.2, C9.1, R3.1: now also TDA2822IC1.7
- net at BT1.1 (+), C14.1, C15.1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: now also TDA2822IC1.2
- net at R5.2: now also C12.1
- net 0 renamed GNDD
- net GNDD: now also C12.2
- new net: D4.1 (K), R2.1
- new net: D4.2 (A), R6.1
- new net GND: C1.2, C10.2, C3.1, C9.2, K1.1 (A), L1.1, R1.2, R3.2, RDA5807FP1.11 (GND), S1.1, S2.1, SW3.2, SW4.2, TDA2822IC1.4, TDA2822IC1.6, Y1.1, Z1.2 (A)
Other:
- moved on the sheet: BT1, C14, R5
