File: 3. ročník/13.10.2025/_autosave-13.10.2025.kicad_sch (KiCad schematic)
At the start: 30 parts, among them J1 Barrel_Jack, SW1 SW_SPST

Commit message: were
Parts:
- added BT1: Battery, symbol Device:Battery
- added SW2, SW3, SW4, SW5: SW_Push, symbol Switch:SW_Push
