File: 3. ročník/FM RADIO RDA/FM RADIO RDA.kicad_sch (KiCad schematic)
At the start: 41 parts, among them J1 Barrel_Jack_Switch, Y1 Crystal

Commit message: HAHA
Parts:
- added H1, H2, H3, H4: MountingHole, MountingHole:MountingHole_2.2mm_M2, symbol Mechanical:MountingHole
- Y1: footprint Crystal:Crystal_AT310_D3.0mm_L10.0mm_Horizontal -> Crystal:Crystal_AT310_D3.0mm_L10.0mm_Vertical
