File: 3. ročník/FM RADIO RDA/FM RADIO RDA.kicad_pcb (KiCad board)
At the start: 2 copper layers, 41 parts, among them J1 Barrel_Jack_Switch, Y1 Crystal

Commit message: HAHA
Parts:
- added H1: MountingHole, MountingHole:MountingHole_2.2mm_M2, F.Cu at (58.5, 86.5)
- added H2: MountingHole, MountingHole:MountingHole_2.2mm_M2, F.Cu at (104.0, 86.5)
- added H3: MountingHole, MountingHole:MountingHole_2.2mm_M2, F.Cu at (104.0, 132.0)
- added H4: MountingHole, MountingHole:MountingHole_2.2mm_M2, F.Cu at (58.5, 131.5)
- Y1: footprint Crystal:Crystal_AT310_D3.0mm_L10.0mm_Horizontal -> Crystal:Crystal_AT310_D3.0mm_L10.0mm_Vertical
- moved RDA5807FP1 76.8 mm to (198.7, 81.9), turned to 90 degrees
- moved ANT1 61.6 mm to (57.0, 74.0)
- moved LS1 48.4 mm to (117.0, 98.3), turned to 90 degrees
- moved S3 35.0 mm to (157.6, 69.2)
- moved S4 35.0 mm to (168.2, 69.2)
- moved S1 21.2 mm to (192.6, 69.2)
- moved S2 21.2 mm to (203.2, 69.2)
- moved C1 20.2 mm to (182.5, 74.0)
- moved C2 20.2 mm to (182.5, 70.0)
- moved L1 12.4 mm to (179.0, 86.5)
- moved D1 11.0 mm to (122.5, 123.8)
- moved R4 10.7 mm to (122.5, 116.3)
- moved R6 9.01 mm to (127.5, 108.8)
- moved L3 8.79 mm to (192.5, 93.5), turned to 180 degrees
- moved R5 8.67 mm to (133.0, 95.2)
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Routing:
- net (no net): vias 2 -> 6
Other:
- board text added: "R8 0"
- board text added: "R9 0"
- board text added: "Speaker"

Commit message: Jasads
Parts:
- moved R6 8.18 mm to (131.9, 101.9)
- moved R5 7.49 mm to (127.0, 99.7)
- moved C1 7.43 mm to (185.0, 81.0), turned to 180 degrees
- moved C2 6.00 mm to (182.5, 76.0)
Routing:
- net Net-(3.7V1-+): track 0.00 -> 149.5 mm
- net Net-(ANT1-A): track 0.00 -> 126.0 mm
- net GND: track 0.00 -> 27.6 mm, vias 0 -> 3
- net Net-(3.7V1--): track 0.00 -> 25.1 mm
- net Net-(D2-K): track 0.00 -> 16.0 mm
- net Net-(C5-Pad1): track 0.00 -> 9.96 mm
- net Net-(C4-Pad1): track 0.00 -> 8.84 mm
- net Net-(C1-Pad1): vias 0 -> 1
- net GNDD: vias 0 -> 1
- net (no net): vias 6 -> 1
